File: MCM-81339-PWR.kicad_sch (KiCad schematic)
At the start: 22 parts, among them J10 694108301002, U1 AZ1117CR-3.3TRG1, U2 LMR16006YQ

Commit message: final version v1.4
* Update: cleanup fabrication layer and placement drawing
* Update: change J6,J7 into J11
Parts:
- L1: footprint Melexis:HPC4018NF-Series -> extra:HPC4018NF-Series
Changed lines of the file:
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@@
 			)
 		)
-		(property "Footprint" "Melexis:HPC4018NF-Series"
+		(property "Footprint" "extra:HPC4018NF-Series"
 			(at 146.05 81.28 0)
 			(effects

Commit message: prepare next devs
Other:
- company: (none) -> Melexis
- title: (none) -> MCM-81339
Changed lines of the file:
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@@
 	(generator_version "9.0")
 	(paper "A4")
+	(title_block
+		(title "MCM-81339")
+		(date "2026-01-28")
+		(rev "v1.5")
+		(company "Melexis")
+	)
 	(junction
 		(at 156.21 81.28)
