File: MCM-81339-SLPWR.kicad_sch (KiCad schematic)
At the start: 17 parts, among them J2 Conn_01x02, U4 VN7040ASTR

Commit message: prepare next devs
Other:
- company: (none) -> Melexis
- title: (none) -> MCM-81339
Changed lines of the file:
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@@
 	(generator_version "9.0")
 	(paper "A4")
+	(title_block
+		(title "MCM-81339")
+		(date "2026-01-28")
+		(rev "v1.5")
+		(company "Melexis")
+	)
 	(junction
 		(at 168.91 90.17)
