File: MCM-81339.kicad_sch (KiCad schematic)
At the start: 5 parts

Commit message: final pcb layout
Parts:
- FID1, FID2, FID3: footprint Fiducial:Fiducial_0.5mm_Mask1mm -> Fiducial:Fiducial_0.75mm_Mask1.5mm
Changed lines of the file:
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@@
       (effects (font (size 1.27 1.27)) (justify left))
     )
-    (property "Footprint" "Fiducial:Fiducial_0.5mm_Mask1mm" (at 138.43 120.65 0)
+    (property "Footprint" "Fiducial:Fiducial_0.75mm_Mask1.5mm" (at 138.43 120.65 0)
       (effects (font (size 1.27 1.27)) hide)
     )
@@
       (effects (font (size 1.27 1.27)) (justify left))
     )
-    (property "Footprint" "Fiducial:Fiducial_0.5mm_Mask1mm" (at 124.46 120.65 0)
+    (property "Footprint" "Fiducial:Fiducial_0.75mm_Mask1.5mm" (at 124.46 120.65 0)
       (effects (font (size 1.27 1.27)) hide)
     )
@@
       (effects (font (size 1.27 1.27)) (justify left))
     )
-    (property "Footprint" "Fiducial:Fiducial_0.5mm_Mask1mm" (at 110.49 120.65 0)
+    (property "Footprint" "Fiducial:Fiducial_0.75mm_Mask1.5mm" (at 110.49 120.65 0)
       (effects (font (size 1.27 1.27)) hide)
     )

Commit message: prepare next devs
Other:
- company: (none) -> Melexis
- title: (none) -> MCM-81339
Changed lines of the file:
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@@
 	(generator_version "9.0")
 	(paper "A4")
+	(title_block
+		(title "MCM-81339")
+		(date "2026-01-28")
+		(rev "v1.5")
+		(company "Melexis")
+	)
 	(symbol
 		(lib_id "Mechanical:Fiducial")
